File: draft-board/draft-board.kicad_sch (KiCad schematic)
At the start: 1 part, among them U1 LM3150MH

Commit message: Buck and LDO
Parts:
- removed U1: LM3150MH, LM3150MH:SOP65P640X110-15N, symbol LM3150MH:LM3150MH
- added C1: 22u, symbol Device:C
- added C10, C9: 100n, symbol Device:C
- added C2, C3: 4.7u, symbol Device:C
- added C4: 88u, symbol Device:C
- added C5, C6, C7: 1u, symbol Device:C
- added C8: 10n, symbol Device:C
- added D1: DSS34, symbol Device:D_Shockley
- added L1: 1.5uH, symbol Device:L
- added R1: 2M, symbol Device:R
- added R2: 200k, symbol Device:R
- added R3: 3.3, symbol Device:R
- added R4: 100k, symbol Device:R
- added U1: NB679GD-Z, NB679GD-Z:VREG_TPS51386RJNR, symbol nb679gd-z:NB679GD-Z
- added U2: RS3236, Package_TO_SOT_SMD:SOT-23-5, symbol rs3236:RS3236
Connections:
- new net: C5.1, R4.2, U1.9 (VCC)
- new net: R1.2, R2.1, U1.11 (EN)
- new net: C3.2, L1.1, U1.7 (SW)
- new net: R3.1, U1.8 (BST)
- new net: C3.1, R3.2
- new net: C8.1, U2.4 (BP)
- new net: R4.1, U1.3 (PG)
- new net: C2.1, U1.6 (LDO)
- new net +24V: C1.1, R1.1, U1.1 (Vin)
- new net +3.3V: C10.1, C7.1, D1.2 (A), U2.5 (OUT)
- new net +5V: C4.1, C6.1, C9.1, D1.1 (K), L1.2, U1.5 (VOUT), U2.1 (IN), U2.3 (EN)
- new net GND: C1.2, C10.2, C2.2, C4.2, C5.2, C6.2, C7.2, C8.2, C9.2, R2.2, U1.10 (AGND), U1.2 (PGND)
- no-connect marks 2 -> 0
Other:
- note added: "24V-5V Buck"
- note added: "3.3 LDO"

Commit message: start layout
Parts:
- removed C4: 88u, symbol Device:C
- removed D1: DSS34, symbol Device:D_Shockley
- removed U2: RS3236, Package_TO_SOT_SMD:SOT-23-5, symbol rs3236:RS3236
- added C11: 33u, Capacitor_SMD:CP_Elec_6.3x7.7, symbol Device:C
- added D1, D2: D_TVS, Diode_SMD:D_SMA, symbol Device:D_TVS
- added F1: Fuse, Fuse:Fuseholder_Cylinder-5x20mm_Bulgin_FX0457_Horizontal_Closed, symbol Device:Fuse
- added H1, H2, H3, H4: MountingHole, MountingHole:MountingHole_3.2mm_M3_DIN965_Pad, symbol Mechanical:MountingHole
- added J1: 24VIN, Connector_AMASS:AMASS_XT60-F_1x02_P7.20mm_Vertical, symbol Connector_Generic:Conn_01x02
- added J2, J3: 24VOUT, Connector_AMASS:AMASS_XT30U-F_1x02_P5.0mm_Vertical, symbol Connector_Generic:Conn_01x02
- added J4: 5VOUT_GH, Connector_JST:JST_GH_BM02B-GHS-TBT_1x02-1MP_P1.25mm_Vertical, symbol Connector_Generic:Conn_01x02
- added J5: 5VOUT_XT30, Connector_AMASS:AMASS_XT30U-F_1x02_P5.0mm_Vertical, symbol Connector_Generic:Conn_01x02
- added K1: SLC-24VDC-SL-C, Relay_THT:Relay_SPDT_RAYEX-L90S, symbol Relay:Relay_SPDT
- added R6: 200k, Resistor_SMD:R_1206_3216Metric, symbol Device:R
- added SW1: SW_SPST, Button_Switch_THT:SW_DIP_SPSTx01_Piano_10.8x4.1mm_W7.62mm_P2.54mm, symbol Switch:SW_SPST
- C1: footprint (none) -> Capacitor_SMD:CP_Elec_6.3x7.7
- C10, C9: value 100n -> 47u; footprint (none) -> Capacitor_SMD:CP_Elec_6.3x7.7
- C2, C3, C5, R3: footprint (none) -> Capacitor_SMD:C_1206_3216Metric
- C6, C7: value 1u -> 47u; footprint (none) -> Capacitor_SMD:CP_Elec_6.3x7.7
- C8: value 10n -> 47u; footprint (none) -> Capacitor_SMD:CP_Elec_6.3x7.7
- L1: footprint (none) -> Inductor_SMD:L_Chilisin_BMRx00060630
- R1, R2, R4: footprint (none) -> Resistor_SMD:R_1206_3216Metric
Connections:
- net +24V: now also C6.1, C7.1, F1.2, K1.11
- net +5V: now also C10.1, C8.1, C11.1, J4.1 (Pin_1), J5.2 (Pin_2); no longer C6.1
- net GND: now also C11.2, J1.1 (Pin_1), J2.1 (Pin_1), J3.1 (Pin_1), J4.2 (Pin_2), J5.1 (Pin_1), K1.A1
- removed net +3.3V: C10.1, C7.1
- new net: D1.1 (A1), D2.1 (A1), F1.1
- new net: R6.2, SW1.1 (A)
- new net: K1.A2, SW1.2 (B)
- new net 24VDC: J1.2 (Pin_2), K1.14, R6.1
- new net 24VOUT: D1.2 (A2), D2.2 (A2), J2.2 (Pin_2), J3.2 (Pin_2)
- no-connect marks 0 -> 1
Other:
- note added: "Connectors"
- note added: "Relay"
- note removed: "3.3 LDO"
- moved on the sheet: C1, C2, C3, C5, L1, R1, R2, R3, R4, U1

Commit message: Finished layout
Parts:
- added C12, C4: 22u, Capacitor_SMD:C_1206_3216Metric, symbol Device:C
- added D3, D4, D5, D6: LED, LED_SMD:LED_0603_1608Metric, symbol Device:LED
- added R5, R7, R8, R9: 100k, Resistor_SMD:R_0603_1608Metric, symbol Device:R
- C2, C3, C5: footprint Capacitor_SMD:C_1206_3216Metric -> Capacitor_SMD:C_0603_1608Metric
- F1: footprint Fuse:Fuseholder_Cylinder-5x20mm_Bulgin_FX0457_Horizontal_Closed -> Fuse:Fuseholder_Cylinder-5x20mm_Stelvio-Kontek_PTF78_Horizontal_Open
- R1, R2, R4, R6: footprint Resistor_SMD:R_1206_3216Metric -> Resistor_SMD:R_0603_1608Metric
- R3: footprint Capacitor_SMD:C_1206_3216Metric -> Resistor_SMD:R_0603_1608Metric
- SW1: footprint Button_Switch_THT:SW_DIP_SPSTx01_Piano_10.8x4.1mm_W7.62mm_P2.54mm -> Button_Switch_THT:SW_DIP_SPSTx01_Slide_9.78x4.72mm_W7.62mm_P2.54mm
Connections:
- net +24V: now also R7.1
- net +5V: now also R8.1
- net 24VDC: now also R5.1
- net 24VOUT: now also F1.1, C12.1, C4.1, R9.1
- net GND: now also D1.1 (A1), D2.1 (A1), C12.2, C4.2, D3.1 (K), D4.1 (K), D5.1 (K), D6.1 (K)
- new net: D5.2 (A), R8.2
- new net: D4.2 (A), R7.2
- new net: D6.2 (A), R9.2
- new net: D3.2 (A), R5.2

Commit message: Polished 2nd time
Parts:
- removed J4: 5VOUT_GH, Connector_JST:JST_GH_BM02B-GHS-TBT_1x02-1MP_P1.25mm_Vertical, symbol Connector_Generic:Conn_01x02
- added C13: 47u, Capacitor_SMD:C_0603_1608Metric, symbol Device:C
- added J6: USB_C_Receptacle_USB2.0_16P, Connector_USB:USB_C_Receptacle_GCT_USB4105-xx-A_16P_TopMnt_Horizontal, symbol Connector:USB_C_Receptacle_USB2.0_16P
Connections:
- net +5V: now also C13.2, J6.A4 (VBUS), J6.A9 (VBUS), J6.B4 (VBUS), J6.B9 (VBUS)
- net GND: now also C13.1, J6.A1 (GND), J6.A12 (GND), J6.B1 (GND), J6.B12 (GND), J6.S1 (SHIELD)
- no-connect marks 1 -> 9
Other:
- moved on the sheet: D3, D4, D5, D6, R5, R7, R8, R9

Commit message: Production
Parts:
- removed C13: 47u, Capacitor_SMD:C_0603_1608Metric, symbol Device:C
Changed lines of the file:
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@@
 	)
 	(junction
-		(at 219.71 102.87)
-		(diameter 0)
-		(color 0 0 0 0)
-	)
-	(junction
 		(at 85.09 115.57)
 		(diameter 0)
@@
 	(wire
 		(pts
-			(xy 228.6 102.87) (xy 219.71 102.87)
+			(xy 214.63 102.87) (xy 228.6 102.87)
 		)
 		(stroke
@@
 	(wire
 		(pts
-			(xy 214.63 102.87) (xy 219.71 102.87)
-		)
-		(stroke
-			(width 0)
-			(type default)
-		)
-	)
-	(wire
-		(pts
 			(xy 63.5 49.53) (xy 63.5 48.26)
 		)
@@
 	(symbol
 		(lib_id "Device:C")
-		(at 219.71 99.06 0)
-		(unit 1)
-		(exclude_from_sim no)
-		(in_bom yes)
-		(on_board yes)
-		(dnp no)
-		(fields_autoplaced yes)
-		(property "Reference" "C13"
-			(at 223.52 97.7899 0)
-			(effects
-				(font
-					(size 1.27 1.27)
-				)
-				(justify left)
-			)
-		)
-		(property "Value" "47u"
-			(at 223.52 100.3299 0)
-			(effects
-				(font
-					(size 1.27 1.27)
-				)
-				(justify left)
-			)
-		)
-		(property "Footprint" "Capacitor_SMD:C_0603_1608Metric"
-			(at 220.6752 102.87 0)
-			(effects
-				(font
-					(size 1.27 1.27)
-				)
-				(hide yes)
-			)
-		)
-		(property "Datasheet" "~"
-			(at 219.71 99.06 0)
-			(effects
-				(font
-					(size 1.27 1.27)
-				)
-				(hide yes)
-			)
-		)
-		(property "Description" "Unpolarized capacitor"
-			(at 219.71 99.06 0)
-			(effects
-				(font
-					(size 1.27 1.27)
-				)
-				(hide yes)
-			)
-		)
-		(pin "1"
-		)
-		(pin "2"
-		)
-		(instances
-			(project "draft-board"
-				(path "/760640d5-a24b-4073-8f9e-eae0457f80de"
-					(reference "C13")
-					(unit 1)
-				)
-			)
-		)
-	)
-	(symbol
-		(lib_id "Device:C")
 		(at 109.22 46.99 0)
 		(unit 1)
@@
 					(unit 1)
 				)
-			)
-		)
-	)
-	(symbol
-		(lib_id "power:GND")
-		(at 219.71 95.25 180)
-		(unit 1)
-		(exclude_from_sim no)
-		(in_bom yes)
-		(on_board yes)
-		(dnp no)
-		(fields_autoplaced yes)
-		(property "Reference" "#PWR022"
-			(at 219.71 88.9 0)
-			(effects
-				(font
-					(size 1.27 1.27)
-				)
-				(hide yes)
-			)
-		)
-		(property "Value" "GND"
-			(at 219.71 90.17 0)
-			(effects
-				(font
-					(size 1.27 1.27)
-				)
-			)
-		)
-		(property "Footprint" ""
-			(at 219.71 95.25 0)
-			(effects
-				(font
-					(size 1.27 1.27)
-				)
-				(hide yes)
-			)
-		)
-		(property "Datasheet" ""
-			(at 219.71 95.25 0)
-			(effects
-				(font
-					(size 1.27 1.27)
-				)
-				(hide yes)
-			)
-		)
-		(property "Description" "Power symbol creates a global label with name \"GND\" , ground"
-			(at 219.71 95.25 0)
-			(effects
-				(font
-					(size 1.27 1.27)
-				)
-				(hide yes)
-			)
-		)
-		(pin "1"
-		)
-		(instances
-			(project ""
-				(path "/760640d5-a24b-4073-8f9e-eae0457f80de"
-					(reference "#PWR022")
-					(unit 1)
-				)
